File: USBtoTTL_HW/USBtoTTL.kicad_pcb (KiCad board)
At the start: 4 copper layers, 25 x 15 mm, 33 parts, among them J1 Socket, J2 USB_C_Receptacle_USB2.0, U1 RT9013-3V3, U2 BD2243G-GTR, U3 CP2104, U4 ESD-BDFN1710A054U

Commit message: 修复一些bug
Parts:
- removed JP2: Jumper_NO_Small, My_Library:JUMP_OPEN_2P_0.3MMx0.5MM
- added R7: 5.1K, Resistor_SMD:R_0402_1005Metric, F.Cu at (66.6, 69.2)
- D1: value OLOAD -> PWR
- D2: value TXD -> OLOAD
- D3: value RXD -> TXD
- D4: value PWR -> RXD
- JP1: value Jumper_NO_Small -> Jump
- R4: value 10K -> 1K
- R6: value 10K -> 5.1K
- moved D4 9.57 mm to (78.9, 68.9), turned to 90 degrees
- moved R5 6.77 mm to (70.6, 71.9)
- moved R4 6.58 mm to (70.8, 64.4)
- moved D2 5.73 mm to (73.8, 63.8), turned to 0 degrees
- moved C1 5.17 mm to (61.7, 61.5), turned to 180 degrees
- moved D1 2.86 mm to (73.8, 60.9)
- moved R6 2.84 mm to (66.6, 66.4)
- moved C3 2.72 mm to (74.3, 71.2), turned to 0 degrees
- moved C4 2.18 mm to (71.2, 73.6), turned to -90 degrees
- moved D3 2.01 mm to (78.9, 67.1), turned to -90 degrees
- moved R1 1.17 mm to (72.2, 73.6), turned to -90 degrees
- moved C9 1.00 mm to (75.3, 67.8), turned to 90 degrees
- moved U3 0.84 mm to (71.3, 67.8)
- moved U2 0.66 mm to (70.7, 62.1)
- moved C7 0.38 mm to (67.7, 73.1)
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Connections:
- D1 pad 1: Net-(D1-Pad1) -> GND
- D2 pad 1: /CP_TXD -> Net-(D2-Pad1)
- D3 pad 1: /CP_RXD -> /CP_TXD
- D3 pad 2: Net-(RN1-Pad2) -> Net-(D3-Pad2)
- D4 pad 1: GND -> /CP_RXD
- D4 pad 2: Net-(RN1-Pad4) -> Net-(D4-Pad2)
- JP1 pad 1: +5V -> Net-(JP1-Pad1)
- JP1 pad 2: Net-(JP1-Pad2) -> +3V3
- R4 pad 1: +5V -> VBUS
- R4 pad 2: Net-(R4-Pad2) -> Net-(D2-Pad2)
- R5 pad 1: Net-(J2-PadA5) -> +5V
- R5 pad 2: GND -> Net-(R5-Pad2)
- R6 pad 1: Net-(J2-PadB5) -> Net-(J2-PadA5)
- RN1 pad 1: Net-(D1-Pad2) -> unconnected-(RN1-Pad1)
- RN1 pad 2: Net-(RN1-Pad2) -> Net-(D4-Pad2)
- RN1 pad 3: Net-(D2-Pad2) -> Net-(D3-Pad2)
- RN1 pad 4: Net-(RN1-Pad4) -> Net-(D1-Pad2)
- U2 pad 4: Net-(D1-Pad1) -> Net-(D2-Pad1)
- U3 pad 5: unconnected-(U3-Pad5) -> Net-(JP1-Pad1)
- U3 pad 6: Net-(JP2-Pad1) -> Net-(JP1-Pad1)
- U3 pad 7: Net-(JP1-Pad2) -> +5V
- U3 pad 9: Net-(R4-Pad2) -> Net-(R5-Pad2)
Routing:
- net GND: track 55.3 -> 0.00 mm, vias 44 -> 0
- net +5V: track 43.1 -> 0.00 mm, vias 14 -> 0
- net VBUS: track 37.2 -> 0.00 mm, vias 6 -> 0
- net /CP_~DTR: track 23.3 -> 0.00 mm, vias 4 -> 0
- net /CP_RXD: track 16.2 -> 0.00 mm, vias 3 -> 0
- net /CP_TXD: track 14.8 -> 0.00 mm, vias 3 -> 0
- net Net-(JP2-Pad1): track 12.7 -> 0.00 mm, vias 2 -> 0
- net +3V3: track 12.3 -> 0.00 mm, vias 3 -> 0
- net Net-(RN1-Pad4): track 9.03 -> 0.00 mm, vias 2 -> 0
- net Net-(D1-Pad2): track 7.77 -> 0.00 mm, vias 2 -> 0
- net Net-(J2-PadA7): track 7.50 -> 0.00 mm
- net Net-(J2-PadA6): track 6.20 -> 0.00 mm, vias 2 -> 0
- net Net-(TP2-Pad1): track 1.90 -> 0.00 mm, vias 1 -> 0
- net Net-(TP1-Pad1): track 1.90 -> 0.00 mm, vias 1 -> 0
- net Net-(D2-Pad2): track 1.87 -> 0.00 mm
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