File: USBtoTTL_HW/USBtoTTL.kicad_sch (KiCad schematic)
At the start: 32 parts, among them J1 Socket, J2 USB_C_Receptacle_USB2.0, U1 RT9013-3V3, U2 BD2243G-GTR, U3 CP2104, U4 ESD-BDFN1710A054U

Commit message: 更新README.md
Other:
- company: (none) -> TurboStudio
- title: (none) -> USBtoTTL
Changed lines of the file:
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@@
 (kicad_sch (version 20211123) (generator eeschema)
   (paper "A4")
+  (title_block
+    (title "USBtoTTL")
+    (date "2022-04-27")
+    (company "TurboStudio")
+    (comment 1 "Design by CubeLine")
+  )
   (junction (at 74.93 104.14) (diameter 0) (color 0 0 0 0)
   )

Commit message: 修复一些bug
Parts:
- removed JP1: Jumper_NO_Small, My_Library:JUMP_OPEN_2P_0.3MMx0.5MM, symbol Device:Jumper_NO_Small
- added R4: 1K, Resistor_SMD:R_0402_1005Metric, symbol Device:R
- JP1: renamed from JP2; value Jumper_NO_Small -> Jump
- R6: renamed from R5; value 10K -> 5.1K
- R7: renamed from R6; value 10K -> 5.1K
- renumbered D4 to D1, D1 to D2, D2 to D3, D3 to D4, R4 to R5
Connections:
- net +5V: now also U3.7 (REGIN)
- net VBUS: now also R4.1
- net at RN1.1 (R1.1): no longer D2.2 (A)
- net at U3.5 (VIO): now also JP1.1, U3.6 (VDD)
- new net: D2.2 (A), R4.2
- no-connect marks 4 -> 5
Other:
- moved on the sheet: D1, D2, JP1, RN1
